Commit message: synced with kortex desc

File: src/feeding_deployment/assets/urdf/feeding_tool/feeding_tool.urdf (robot description, URDF)
Before this commit: robot flair_feeding_utensil, 5 links, 4 joints
Links:
- removed link feeding_utensil_tip
- removed link forque_tip
- added link feeding_tool_tip, mass 0
- added link fork_tip, mass 0
- link forkbase: mass 0.097534 -> 0.072775; geometry collision mesh filename=tool_base.stl; visual mesh filename=tool_base.stl
- link forkpitch: mass 0.019491 -> 0.072775; geometry collision mesh filename=tool_pitch.stl; visual mesh filename=tool_pitch.stl
- link forkroll: geometry collision mesh filename=tool_roll.stl; visual mesh filename=tool_roll.stl
Joints:
- removed joint joint_feeding_utensil_tip
- added joint joint_feeding_tool_tip: type fixed, parent forkroll, child feeding_tool_tip, origin xyz=0.13 0.0 0.0 rpy=0 0 0, axis 0 0 0, limit lower=0 upper=0 effort=2000 velocity=1
- joint forkpitch_joint: axis 0 1 0 -> 0 0 -1; origin xyz=0.0395 0 0 rpy=0 0 0 -> xyz=0.11 0.0 -0.087 rpy=0 0 0
- joint forkroll_joint: origin xyz=0.045083 0 0 rpy=0 0 0 -> xyz=0.0151 0.0 0.0095   rpy=-1.570796 0 0
- joint joint_fork_tip: child forque_tip -> fork_tip; parent feeding_utensil_tip -> feeding_tool_tip

File: src/feeding_deployment/assets/urdf/flair_feeding_tool/feeding_tool.urdf (robot description, URDF)
Before this commit: robot feeding_utensil, 5 links, 4 joints
Links:
- removed link feeding_utensil_tip
- removed link forque_tip
- added link feeding_tool_tip, mass 0
- added link fork_tip, mass 0
- link forkbase: mass 0.072775 -> 0.097534; geometry collision mesh filename=tool_base.stl; visual mesh filename=tool_base.stl
- link forkpitch: mass 0.072775 -> 0.019491; geometry collision mesh filename=tool_pitch.stl; visual mesh filename=tool_pitch.stl
- link forkroll: geometry collision mesh filename=tool_roll.stl; visual mesh filename=tool_roll.stl
Joints:
- removed joint joint_feeding_utensil_tip
- added joint joint_feeding_tool_tip: type fixed, parent forkroll, child feeding_tool_tip, origin xyz=0.095 0.00 0.00 rpy=0 0 0, axis 0 0 0, limit lower=0 upper=0 effort=2000 velocity=1
- joint forkpitch_joint: axis 0 0 -1 -> 0 1 0; origin xyz=0.11 0.0 -0.087 rpy=0 0 0 -> xyz=0.0395 0 0 rpy=0 0 0
- joint forkroll_joint: origin xyz=0.0151 0.0 0.0095   rpy=-1.570796 0 0 -> xyz=0.045083 0 0 rpy=0 0 0
- joint joint_fork_tip: child forque_tip -> fork_tip; parent feeding_utensil_tip -> feeding_tool_tip

Commit message: wpi

File: src/feeding_deployment/assets/urdf/feeding_tool/feeding_tool.urdf (robot description, URDF)
Before this commit: robot feeding_tool, 5 links, 4 joints
Joints:
- joint joint_feeding_tool_tip: origin xyz=0.13 0.0 0.0 rpy=0 0 0 -> xyz=0.097 0.00 -0.002 rpy=0 0 0

Commit message: wip

File: src/feeding_deployment/assets/urdf/feeding_tool/feeding_tool.urdf (robot description, URDF)
Before this commit: robot feeding_utensil, 5 links, 4 joints
Links:
- removed link feeding_utensil_tip
- removed link forque_tip
- added link feeding_tool_tip, mass 0
- added link fork_tip, mass 0
- link forkbase: geometry collision mesh filename=tool_base.stl; visual mesh filename=tool_base.stl
- link forkpitch: geometry collision mesh filename=tool_pitch.stl; visual mesh filename=tool_pitch.stl
- link forkroll: geometry collision mesh filename=tool_roll.stl; visual mesh filename=tool_roll.stl
Joints:
- removed joint joint_feeding_utensil_tip
- added joint joint_feeding_tool_tip: type fixed, parent forkroll, child feeding_tool_tip, origin xyz=0.097 0.00 -0.002 rpy=0 0 0, axis 0 0 0, limit lower=0 upper=0 effort=2000 velocity=1
- joint joint_fork_tip: child forque_tip -> fork_tip; parent feeding_utensil_tip -> feeding_tool_tip
