Commit message: using multiple drink urdfs + disabled joint following error

File: src/feeding_deployment/robot_controller/hack_gen3_robotiq_2f_85_drink_6.urdf (robot description, URDF)
Before this commit: robot gen3_robotiq_2f_85_feeding, 14 links, 13 joints
Links:
- link robotiq_arg2f_base_link: mass 1.9 -> 1.7
